File: hardware/pcb/02_FPGA_Core.kicad_sch (KiCad schematic)
At the start: 0 parts

Commit message: feat: add power rails to the fpga gowin arora v family symbol
Parts:
- added C20, C21, C22, C23, C24, C25, C26, C27, C28, C29, C30, C31, C32, C33, C34, C35: 0.1uF, symbol Device:C
- added C36, C37, C38: 10uF, symbol Device:C
- added C39: 1uF, symbol Device:C
- added U4: GW5A-LV25MG121N, symbol symbol-table:GW5A-LV25MG121N
Connections:
- new net +1V2: C20.1, C21.1, C22.1, C23.1, C24.1, C36.1, U4.D9 (VDDDM), U4.E9 (VCC), U4.F4 (VCC), U4.F8 (VCC), U4.K3 (VDD12M)
- new net +2V5: C25.1, C26.1, C27.1, C28.1, C35.1, C37.1, U4.C8 (VDDAM), U4.G3 (VCCX_VDDXM), U4.G6 (VCCX_VDDXM), U4.G9 (VCCX_VDDXM), U4.H3 (VCCX_VDDXM)
- new net +3V3: C29.1, C30.1, C31.1, C32.1, C33.1, C34.1, C38.1, U4.A4 (VCCIO2_3), U4.D2 (VCCIO5_10), U4.D4 (VCCIO4), U4.F10 (VCCIO6_7), U4.J9 (VCCIO0_1)
- new net GND: C20.2, C21.2, C22.2, C23.2, C24.2, C25.2, C26.2, C27.2, C28.2, C29.2, C30.2, C31.2, C32.2, C33.2, C34.2, C35.2, C36.2, C37.2, C38.2, C39.2, U4.B4 (VSS), U4.C5 (VSS), U4.C7 (VSS), U4.C9 (VSS), U4.D3 (VEFUSE), U4.F11 (VSS), U4.F3 (VSS), U4.F9 (VSS), U4.H6 (VSS), U4.H9 (VSS), U4.J3 (VSS)
- new net VCCLDO: C39.1, U4.J6 (VCCLDO)
- no-connect marks 0 -> 2

Commit message: feat: wtv i have done as of yet
Parts:
- added U6: GW5A-LV25MG121N, symbol symbol-table:GW5A-LV25MG121N
Connections:
- new net FPGA_DONE: U6.D7 (IOB64A/DONE)
- new net FPGA_MODE0: U6.VCCIO_MODE0 (IOB62B/MODE0)
- new net FPGA_MODE1: U6.GND_MODE1 (IOB52A/MODE1)
- new net FPGA_PUDC_B: U6.GND_PUDC (IOT29A/PUDC_B)
- new net FPGA_READY: U6.E8 (IOB37A/READY)
- new net FPGA_RECONFIG_N: U6.D8 (IOB1A/RECONFIG_N)
- new net JTAG_TCK: U6.C1 (IOR1A/TCK)
- new net JTAG_TDI: U6.A3 (IOR1B/TDI)
- new net JTAG_TDO: U6.A2 (IOR3B/TDO)
- new net JTAG_TMS: U6.B1 (IOR3A/TMS)

Commit message: feat: fix sheet 2
Parts:
- added D1: Green, symbol Device:LED
- added R7, R9: 10k, symbol Device:R
- added R8: 1k, symbol Device:R
- renumbered U6 to U4
Connections:
- net +3V3: now also R7.1, R8.1, R9.1
- net FPGA_DONE: now also D1.2 (A), R8.2
- net FPGA_READY: now also R9.2
- net FPGA_RECONFIG_N: now also R7.2
- net GND: now also D1.1 (K)
- removed net FPGA_MODE0: U4.VCCIO_MODE0 (IOB62B/MODE0)
- removed net FPGA_MODE1: U4.GND_MODE1 (IOB52A/MODE1)
- removed net FPGA_PUDC_B: U4.GND_PUDC (IOT29A/PUDC_B)
- no-connect marks 2 -> 14
